Commit message: With Navigation

File: src/simulation_env/models/auto/auto.xacro (robot description, xacro)
@@ -139,3 +139,57 @@
     <joint_properties damping="0.0" friction="0.0"/>
   </joint>
- </robot>
+  <!-- Add a Hokuyo Laser -->
+  <link name="laser_link">
+    <collision>
+      <origin xyz="0 0 0" rpy="0 0 0"/>
+      <geometry>
+		<box size="${x_hokuyo} ${y_hokuyo} ${z_hokuyo}"/>
+      </geometry>
+    </collision>
+    <visual>
+      <origin xyz="0 0 0" rpy="0 0 0"/>
+      <geometry>
+        <!-- <mesh filename="package://rrbot_description/meshes/hokuyo.dae"/> -->
+        <box size="${x_hokuyo} ${y_hokuyo} ${z_hokuyo}"/>
+      </geometry>
+    </visual>
+    <inertial>
+      <mass value="1e-5" />
+      <origin xyz="0 0 0" rpy="0 0 0"/>
+      <inertia ixx="1e-6" ixy="0" ixz="0" iyy="1e-6" iyz="0" izz="1e-6" />
+    </inertial>
+  </link>
+  <joint name="hokuyo_joint" type="fixed">
+    <axis xyz="0 1 0" />
+    <origin xyz="0 0 ${z_chassis/2 + z_hokuyo/2}" rpy="0 0 0"/>
+    <parent link="base_link"/>
+    <child link="laser_link"/>
+  </joint>
+  <!-- Add the camera link -->
+  <link name="camera_link">
+    <collision>
+      <origin xyz="0 0 0" rpy="0 0 0"/>
+      <geometry>
+    <box size="${camera_size} ${camera_size} ${camera_size}"/>
+      </geometry>
+    </collision>
+    <visual>
+      <origin xyz="0 0 0" rpy="0 0 0"/>
+      <geometry>
+    <box size="${camera_size} ${camera_size} ${camera_size}"/>
+      </geometry>
+      <material name="red"/>
+    </visual>
+    <inertial>
+      <mass value="1e-5" />
+      <origin xyz="0 0 0" rpy="0 0 0"/>
+      <inertia ixx="1e-6" ixy="0" ixz="0" iyy="1e-6" iyz="0" izz="1e-6" />
+    </inertial>
+  </link>
+  <joint name="camera_joint" type="fixed">
+    <axis xyz="0 1 0" />
+    <origin xyz="0 0 ${z_hokuyo/2 + camera_size/2}" rpy="0 0 0"/>
+    <parent link="laser_link"/>
+    <child link="camera_link"/>
+  </joint>
+</robot>

File: src/simulation_env/models/auto/parameter.xacro (robot description, xacro)
@@ -13,3 +13,7 @@
   <!-- <xacro:property name="L_wheel" value="${properties['axis_distance']}" /> -->
   <xacro:property name="L_wheel" value="0.1789" />
+  <xacro:property name="x_hokuyo" value="0.1" />
+  <xacro:property name="y_hokuyo" value="0.1" />
+  <xacro:property name="z_hokuyo" value="0.1" />
+  <xacro:property name="camera_size" value="0.05" />
 </robot>
